File: PCB/keyboard.kicad_sch (KiCad schematic)
At the start: 351 parts, among them J1 USB_C_Receptacle_USB2.0_14P, Q1 AO3400A, SW1 SW_Push, U1 AT90USB1286-A, U2 EC11E18244A5, U3 EC11E18244A5, Y1 16MHz

Commit message: Firmware
Connections:
- net col12: now also U1.25 (PD0); no longer U1.17 (PB7)
- net at R8.1: now also U1.17 (PB7); no longer U1.28 (PD3)
Changed lines of the file:
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@@
 	(wire
 		(pts
+			(xy 204.47 331.47) (xy 204.47 367.03)
+		)
+		(stroke
+			(width 0)
+			(type default)
+		)
+	)
+	(wire
+		(pts
 			(xy 325.12 190.5) (xy 325.12 191.77)
 		)
@@
 	(wire
 		(pts
+			(xy 184.15 359.41) (xy 182.88 359.41)
+		)
+		(stroke
+			(width 0)
+			(type default)
+		)
+	)
+	(wire
+		(pts
 			(xy 656.59 250.19) (xy 656.59 240.03)
 		)
@@
 	(wire
 		(pts
+			(xy 204.47 367.03) (xy 222.25 367.03)
+		)
+		(stroke
+			(width 0)
+			(type default)
+		)
+	)
+	(wire
+		(pts
 			(xy 351.79 87.63) (xy 351.79 138.43)
 		)
@@
 	(wire
 		(pts
-			(xy 182.88 367.03) (xy 222.25 367.03)
-		)
-		(stroke
-			(width 0)
-			(type default)
-		)
-	)
-	(wire
-		(pts
 			(xy 165.1 384.81) (xy 156.21 384.81)
 		)
@@
 	(wire
 		(pts
-			(xy 182.88 331.47) (xy 186.69 331.47)
+			(xy 182.88 331.47) (xy 204.47 331.47)
 		)
 		(stroke
@@
 		)
 	)
+	(global_label "col12"
+		(shape input)
+		(at 184.15 359.41 0)
+		(fields_autoplaced yes)
+		(effects
+			(font
+				(size 1.27 1.27)
+			)
+			(justify left)
+		)
+		(property "Intersheetrefs" "${INTERSHEET_REFS}"
+			(at 534.67 375.92 0)
+			(effects
+				(font
+					(size 1.27 1.27)
+				)
+				(hide yes)
+			)
+		)
+	)
 	(global_label "col17"
 		(shape input)
@@
 			(effects
 				(font
-					(size 1.27 1.27)
-				)
-				(hide yes)
-			)
-		)
-	)
-	(global_label "col12"
-		(shape input)
-		(at 186.69 331.47 0)
-		(fields_autoplaced yes)
-		(effects
-			(font
-				(size 1.27 1.27)
-			)
-			(justify left)
-		)
-		(property "Intersheetrefs" "${INTERSHEET_REFS}"
-			(at 537.21 347.98 0)
-			(effects
-				(font

Commit message: PCB
Parts:
- removed C2: 22pF, Capacitor_SMD:C_0805_2012Metric, symbol Device:C_Small
- removed C3: 1uF, Capacitor_SMD:C_0805_2012Metric, symbol Device:C_Small
- removed C4, C5, C6: 0.1uF, Capacitor_SMD:C_0805_2012Metric, symbol Device:C_Small
- removed C7: 10uF, Capacitor_SMD:C_0805_2012Metric, symbol Device:C_Small
- removed Q1: AO3400A, Package_TO_SOT_SMD:SOT-23, symbol Transistor_FET:AO3400A
- removed R1, R6: 10k, Resistor_SMD:R_0805_2012Metric, symbol Device:R_Small
- removed R4, R5: 22, Resistor_SMD:R_0805_2012Metric, symbol Device:R_Small
- removed SW1: SW_Push, random-keyboard-parts:SKQG-1155865, symbol Switch:SW_Push
- removed U1: AT90USB1286-A, Package_QFP:TQFP-64_14x14mm_P0.8mm, symbol MCU_Microchip_AVR:AT90USB1286-A
- removed Y1: 16MHz, Crystal:Crystal_SMD_3225-4Pin_3.2x2.5mm, symbol Device:Crystal_GND24_Small
- added C13, C15, C17: 0.1uF, Capacitor_SMD:C_0402_1005Metric, symbol Device:C_Small
- added C14: 10uF, Capacitor_SMD:C_0402_1005Metric, symbol Device:C_Small
- added C16: 4.7uF, Capacitor_SMD:C_0402_1005Metric, symbol Device:C_Small
- added J2: Conn_01x02, Connector_PinHeader_2.54mm:PinHeader_1x02_P2.54mm_Horizontal, symbol Connector_Generic:Conn_01x02
- added J3: Conn_01x05_Socket, Connector_PinHeader_2.54mm:PinHeader_1x05_P2.54mm_Horizontal, symbol Connector:Conn_01x05_Socket
- added Q2: AO3400A, Package_TO_SOT_SMD:SOT-23, symbol Transistor_FET:AO3400A
- added R1: 1.8k, Capacitor_SMD:C_0805_2012Metric, symbol Device:R
- added SW1: SW_MAIN_PWR, SPST:EG1206A_EWI, symbol Switch:SW_SPST
- added U1: TP4056-42-ESOP8, Package_SO:SOIC-8-1EP_3.9x4.9mm_P1.27mm_EP2.41x3.3mm_ThermalVias, symbol Battery_Management:TP4056-42-ESOP8
- added U4: ~, ProLib_pcs_2025-05-29 (3):LCC-LGA-54_L24.0-W20.5_RF-BM-ND06, symbol ProLib_pcs_2025-05-29 (2):RF-BM-ND06
- added U5: AP2112K-3.3, Package_TO_SOT_SMD:SOT-23-5, symbol Regulator_Linear:AP2112K-3.3
- C1: value 22pF -> 10uF; footprint Capacitor_SMD:C_0805_2012Metric -> Capacitor_SMD:C_0603_1608Metric
- R10, R100, R101, R102, R103, R104, R105, R106, R107, R108, R109, R11, R110, R111, R112, R113, R114, R115, R116, R117, R118, R12, R13, R14, R15, R16, R17, R18, R19, R20, R21, R22, R23, R24, R25, R26, R27, R28, R29, R30, R31, R32, R33, R34, R35, R36, R37, R38, R39, R40, R41, R42, R43, R44, R45, R46, R47, R48, R49, R50, R51, R52, R53, R54, R55, R56, R57, R58, R59, R60, R61, R62, R63, R64, R65, R66, R67, R68, R69, R70, R71, R72, R73, R74, R75, R76, R77, R78, R79, R80, R81, R82, R83, R84, R85, R86, R87, R88, R89, R90, R91, R92, R93, R94, R95, R96, R97, R98, R99: value 120 -> 22
- R7: footprint Resistor_SMD:R_0805_2012Metric -> Resistor_SMD:R_2010_5025Metric
Connections:
- net +5V: now also C1.2, C15.1, C16.1, C17.1, U1.4 (V_{CC}), U1.8 (CE), U4.3 (VDD_HV), U4.4 (VDD_USB); no longer R10.1, R100.1, R101.1, R102.1, R103.1, R104.1, R105.1, R106.1, R107.1, R108.1, R109.1, R11.1, R110.1, R111.1, R112.1, R113.1, R114.1, R115.1, R116.1, R117.1, R118.1, R12.1, R13.1, R14.1, R15.1, R16.1, R17.1, R18.1, R19.1, R20.1, R21.1, R22.1, R23.1, R24.1, R25.1, R26.1, R27.1, R28.1, R29.1, R30.1, R31.1, R32.1, R33.1, R34.1, R35.1, R36.1, R37.1, R38.1, R39.1, R40.1, R41.1, R42.1, R43.1, R44.1, R45.1, R46.1, R47.1, R48.1, R49.1, R50.1, R51.1, R52.1, R53.1, R54.1, R55.1, R56.1, R57.1, R58.1, R59.1, R60.1, R61.1, R62.1, R63.1, R64.1, R65.1, R66.1, R67.1, R68.1, R69.1, R70.1, R71.1, R72.1, R73.1, R74.1, R75.1, R76.1, R77.1, R78.1, R79.1, R80.1, R81.1, R82.1, R83.1, R84.1, R85.1, R86.1, R87.1, R88.1, R89.1, R90.1, R91.1, R92.1, R93.1, R94.1, R95.1, R96.1, R97.1, R98.1, R99.1, VR1.3 (CW)
- net D+: now also U4.6 (D+)
- net D-: now also U4.5 (D-)
- net GND: now also C13.1, C14.1, C15.2, C16.2, C17.2, J2.2 (Pin_2), J3.4 (Pin_4), Q2.2 (S), R1.2, U1.1 (TEMP), U1.3 (GND), U1.9 (EPAD), U5.2 (GND)
- net LED-: now also Q2.3 (D)
- net PC1: now also U4.40 (P0.02)
- net PC2: now also U4.39 (P0.03)
- net PC3: now also U4.48 (P0.05)
- net PC4: now also U4.47 (P0.04)
- net PC5: now also U4.43 (P0.30)
- net PC6: now also U4.42 (P0.29)
- net col0: now also U4.36 (P1.13)
- net col1: now also U4.37 (P1.14)
- net col10: now also U4.26 (P1.02)
- net col11: now also U4.27 (P1.03)
- net col12: now also U4.49 (P0.06)
- net col13: now also U4.50 (P0.07)
- net col14: now also U4.51 (P0.08)
- net col15: now also U4.52 (P1.08)
- net col16: now also U4.44 (P0.31)
- net col17: now also U4.54 (P0.11)
- net col19: now also U4.7 (P0.13)
- net col2: now also U4.38 (P1.15)
- net col20: now also U4.8 (P0.14)
- net col21: now also U4.28 (P1.04)
- net col22: now also U4.29 (P1.05)
- net col4: now also U4.10 (P0.16)
- net col5: now also U4.11 (P0.17)
- net col6: now also U4.16 (P0.22)
- net col7: now also U4.13 (P0.19)
- net col8: now also U4.14 (P0.20)
- net col9: now also U4.15 (P0.21)
- net row0: now also U4.30 (P1.06)
- net row2: now also U4.32 (P1.07)
- net row3: now also U4.53 (P1.09)
- net row4: now also U4.33 (P1.10)
- net row5: now also U4.34 (P1.11)
- net row6: now also U4.35 (P1.12)
- net at R7.2, R8.2: now also Q2.1 (G)
- net at R8.1: now also U4.25 (P1.01)
- net PF0 renamed PC7
- net PC7: now also U4.41 (P0.28)
- new net: R1.1, U1.2 (PROG)
- new net: SW1.1 (A), U1.5 (BAT), U5.1 (VIN), U5.3 (EN)
- new net: J3.2 (Pin_2), U4.22 (SWCLK)
- new net: J3.3 (Pin_3), U4.21 (SWDIO)
- new net: J2.1 (Pin_1), SW1.2 (B)
- new net: U4.55 (NC), U4.56 (NC), U4.57 (NC), U4.58 (NC), U4.59 (NC), U4.60 (NC), U4.61 (NC), U4.62 (NC), U4.63 (NC)
- new net +3.3V: C13.2, C14.2, J3.5 (Pin_5), R10.1, R100.1, R101.1, R102.1, R103.1, R104.1, R105.1, R106.1, R107.1, R108.1, R109.1, R11.1, R110.1, R111.1, R112.1, R113.1, R114.1, R115.1, R116.1, R117.1, R118.1, R12.1, R13.1, R14.1, R15.1, R16.1, R17.1, R18.1, R19.1, R20.1, R21.1, R22.1, R23.1, R24.1, R25.1, R26.1, R27.1, R28.1, R29.1, R30.1, R31.1, R32.1, R33.1, R34.1, R35.1, R36.1, R37.1, R38.1, R39.1, R40.1, R41.1, R42.1, R43.1, R44.1, R45.1, R46.1, R47.1, R48.1, R49.1, R50.1, R51.1, R52.1, R53.1, R54.1, R55.1, R56.1, R57.1, R58.1, R59.1, R60.1, R61.1, R62.1, R63.1, R64.1, R65.1, R66.1, R67.1, R68.1, R69.1, R70.1, R71.1, R72.1, R73.1, R74.1, R75.1, R76.1, R77.1, R78.1, R79.1, R80.1, R81.1, R82.1, R83.1, R84.1, R85.1, R86.1, R87.1, R88.1, R89.1, R90.1, R91.1, R92.1, R93.1, R94.1, R95.1, R96.1, R97.1, R98.1, R99.1, U4.2 (VCC), U5.5 (VOUT), VR1.3 (CW)
- new net Nreset: J3.1 (Pin_1), U4.12 (P0.18)
- new net STBY: U1.6 (~{STDBY}), U4.46 (P0.27)
- new net chrg: U1.7 (~{CHRG}), U4.45 (P0.26)
Other:
- moved on the sheet: F1, J1, R2, R3, U2, U3, VR1
